File: kicad/main/MicroController.sch (KiCad schematic (older format))
At the start: 7 parts, among them P3 MIKROPROG, U1 LM324, U2 PIC16F1779

Commit message: Made more PCB's, finished Display PCB
Parts:
- added C?: 100n, symbol C_Small
- added P?: DISPLAY, symbol CONN_01X20
- added Q?: BC847, symbol Q_NPN_BEC
- added R?: 20, Resistors_SMD:R_0805_HandSoldering, symbol R
- added R?: 4k7, Resistors_SMD:R_0805_HandSoldering, symbol R
- added RV?: 10k, symbol POT_TRIM
Connections:
- net RB7 is gone; now on net RA2: U1.3 (+)
- net +5V: now also C?.1, P?.19 (P19), P?.4 (P4)
- net GND: now also C?.2, P?.3 (P3), Q?.2 (E), RV?.1
- net RB0: now also P?.1 (P1)
- net RB1: now also P?.2 (P2)
- net RB2: now also P?.6 (P6)
- net RB3: now also P?.7 (P7)
- net RB4: now also P?.8 (P8)
- net RB5: now also P?.17 (P17)
- net RC2: now also R?.2; no longer P?.3 (P3)
- net RC3: now also P?.3 (P3)
- net RD0: now also P?.9 (P9)
- net RD1: now also P?.10 (P10)
- net RD2: now also P?.11 (P11)
- net RD3: now also P?.12 (P12)
- net RD4: now also P?.13 (P13)
- net RD5: now also P?.14 (P14)
- net RD6: now also P?.15 (P15)
- net RD7: now also P?.16 (P16)
- new net: P?.18 (P18), RV?.3
- new net: P?.20 (P20), R?.2
- new net: P?.5 (P5), RV?.2
- new net: Q?.1 (B), R?.1
- new net: Q?.3 (C), R?.1
Other:
- note added: "DISPLAY CONNECTOR"
Changed lines of the file:
@@
 Connection ~ 1800 2650
 Text Label 1000 2550 2    60   ~ 0
-RB7
+RA2
 Wire Wire Line
 	1000 2550 1100 2550
@@
 RC1
 Text Label 2400 7000 2    60   ~ 0
-RC2
+RC3
 Wire Wire Line
 	2400 6800 2500 6800
@@
 Wire Wire Line
 	2100 7100 2500 7100
+$Comp
+L CONN_01X20 P?
+U 1 1 59D5FF47
+P 4825 5150
+F 0 "P?" H 4825 6200 50  0000 C CNN
+F 1 "DISPLAY" V 4925 5150 50  0000 C CNN
+F 2 "" H 4825 5150 50  0000 C CNN
+F 3 "" H 4825 5150 50  0000 C CNN
+	1    4825 5150
+	1    0    0    -1
+$EndComp
+Text Label 4525 5000 2    60   ~ 0
+RD0
+Text Label 4525 5100 2    60   ~ 0
+RD1
+Text Label 4525 5200 2    60   ~ 0
+RD2
+Text Label 4525 5300 2    60   ~ 0
+RD3
+Text Label 4525 5400 2    60   ~ 0
+RD4
+Text Label 4525 5500 2    60   ~ 0
+RD5
+Text Label 4525 5600 2    60   ~ 0
+RD6
+Text Label 4525 5700 2    60   ~ 0
+RD7
+Text Label 4525 4200 2    60   ~ 0
+RB0
+Text Label 4525 4300 2    60   ~ 0
+RB1
+Text Label 4525 4700 2    60   ~ 0
+RB2
+Text Label 4525 4800 2    60   ~ 0
+RB3
+Text Label 4525 4900 2    60   ~ 0
+RB4
+Text Label 4525 5800 2    60   ~ 0
+RB5
+$Comp
+L +5V #PWR?
+U 1 1 59D607C5
+P 4125 4250
+F 0 "#PWR?" H 4125 4100 50  0001 C CNN
+F 1 "+5V" H 4125 4390 50  0000 C CNN
+F 2 "" H 4125 4250 50  0000 C CNN
+F 3 "" H 4125 4250 50  0000 C CNN
+	1    4125 4250
+	1    0    0    -1
+$EndComp
+$Comp
+L GND #PWR?
+U 1 1 59D60849
+P 4175 6150
+F 0 "#PWR?" H 4175 5900 50  0001 C CNN
+F 1 "GND" H 4175 6000 50  0000 C CNN
+F 2 "" H 4175 6150 50  0000 C CNN
+F 3 "" H 4175 6150 50  0000 C CNN
+	1    4175 6150
+	1    0    0    -1
+$EndComp
+Wire Wire Line
+	4175 6150 4175 4400
+Wire Wire Line
+	4175 4400 4625 4400
+Wire Wire Line
+	4125 4250 4125 4500
+Wire Wire Line
+	4125 4500 4625 4500
+$Comp
+L C_Small C?
+U 1 1 59D60C67
+P 3925 4500
+F 0 "C?" H 3935 4570 50  0000 L CNN
+F 1 "100n" H 3935 4420 50  0000 L CNN
+F 2 "" H 3925 4500 50  0000 C CNN
+F 3 "" H 3925 4500 50  0000 C CNN
+	1    3925 4500
+	1    0    0    -1
+$EndComp
+Wire Wire Line
+	3925 4400 3925 4350
+Wire Wire Line
+	3475 4350 4125 4350
+Connection ~ 4125 4350
+Wire Wire Line
+	3925 4600 3925 4650
+Wire Wire Line
+	3775 4650 4175 4650
+Connection ~ 4175 4650
+$Comp
+L POT_TRIM RV?
+U 1 1 59D60E6A
+P 3775 4850
+F 0 "RV?" V 3600 4850 50  0000 C CNN
+F 1 "10k" V 3675 4850 50  0000 C CNN
+F 2 "" H 3775 4850 50  0000 C CNN
+F 3 "" H 3775 4850 50  0000 C CNN
+	1    3775 4850
+	1    0    0    -1
+$EndComp
+Wire Wire Line
+	3775 4700 3775 4650
+Connection ~ 3925 4650
+Wire Wire Line
+	3775 5000 3775 5900
+Wire Wire Line
+	3775 5900 4625 5900
+Wire Wire Line
+	3925 4850 4275 4850
+Wire Wire Line
+	4275 4850 4275 4600
+Wire Wire Line
+	4275 4600 4625 4600
+Wire Wire Line
+	4625 6000 3475 6000
+Wire Wire Line
+	3475 6000 3475 4350
+Connection ~ 3925 4350
+$Comp
+L Q_NPN_BEC Q?
+U 1 1 59D613CD
+P 4475 6700
+F 0 "Q?" H 4675 6750 50  0000 L CNN
+F 1 "BC847" H 4675 6650 50  0000 L CNN
+F 2 "" H 4675 6800 50  0000 C CNN
+F 3 "" H 4475 6700 50  0000 C CNN
+	1    4475 6700
+	1    0    0    -1
+$EndComp
+Wire Wire Line
+	4575 6100 4625 6100
+$Comp
+L R R?
+U 1 1 59D614FF
+P 4575 6300
+F 0 "R?" V 4655 6300 50  0000 C CNN
+F 1 "20" V 4575 6300 50  0000 C CNN
+F 2 "Resistors_SMD:R_0805_HandSoldering" V 4505 6300 50  0001 C CNN
+F 3 "" H 4575 6300 50  0000 C CNN
+	1    4575 6300
+	-1   0    0    1
+$EndComp
+Wire Wire Line
+	4575 6150 4575 6100
+Wire Wire Line
+	4575 6500 4575 6450
+$Comp
+L R R?
+U 1 1 59D619A5
+P 4075 6700
+F 0 "R?" V 4155 6700 50  0000 C CNN
+F 1 "4k7" V 4075 6700 50  0000 C CNN
+F 2 "Resistors_SMD:R_0805_HandSoldering" V 4005 6700 50  0001 C CNN
+F 3 "" H 4075 6700 50  0000 C CNN
+	1    4075 6700
+	0    1    1    0
+$EndComp
+Wire Wire Line
+	4225 6700 4275 6700
+$Comp
+L GND #PWR?
+U 1 1 59D61D4B
+P 4575 6950
+F 0 "#PWR?" H 4575 6700 50  0001 C CNN
+F 1 "GND" H 4575 6800 50  0000 C CNN
+F 2 "" H 4575 6950 50  0000 C CNN
+F 3 "" H 4575 6950 50  0000 C CNN
+	1    4575 6950
+	1    0    0    -1
+$EndComp
+Wire Wire Line
+	4575 6950 4575 6900
+Wire Wire Line
+	4525 4200 4625 4200
+Wire Wire Line
+	4525 4300 4625 4300
+Wire Wire Line
+	4525 4700 4625 4700
+Wire Wire Line
+	4525 4800 4625 4800
+Wire Wire Line
+	4525 4900 4625 4900
+Wire Wire Line
+	4525 5000 4625 5000
+Wire Wire Line
+	4525 5100 4625 5100
+Wire Wire Line
+	4525 5200 4625 5200
+Wire Wire Line
+	4525 5300 4625 5300
+Wire Wire Line
+	4525 5400 4625 5400
+Wire Wire Line
+	4525 5500 4625 5500
+Wire Wire Line
+	4525 5600 4625 5600
+Wire Wire Line
+	4525 5700 4625 5700
+Wire Wire Line
+	4525 5800 4625 5800
+Text Label 3875 6700 2    60   ~ 0
+RC2
+Wire Wire Line
+	3875 6700 3925 6700
+Wire Notes Line
+	2950 3750 5550 3750
+Wire Notes Line
+	5550 7250 5550 3750
+Wire Notes Line
+	2950 7250 5550 7250
+Wire Notes Line
+	2950 7250 2950 3750
+Text Notes 4575 3875 0    60   ~ 0
+DISPLAY CONNECTOR
 $EndSCHEMATC
